File: Avionics-SolarPanels.kicad_pcb (KiCad board)
At the start: 4 copper layers, 82 x 100 mm, 213 parts, among them J1 200528-0100, J2 200528-0100, Q1 NX3008NBKS, Q10 MBT2222ADW1T1, Q11 NX3008NBKS, Q12 MBT2222ADW1T1, Q13 NX3008NBKS, Q14 MBT2222ADW1T1, Q15 NX3008NBKS, Q16 MBT2222ADW1T1, Q2 MBT2222ADW1T1, Q3 NX3008NBKS, Q4 MBT2222ADW1T1, Q5 NX3008NBKS, Q6 MBT2222ADW1T1, Q7 NX3008NBKS, Q8 MBT2222ADW1T1, Q9 NX3008NBKS, U1 OPT4003DNPRQ1, U10 NCV891330PD50R2G, U11 LTC4376CDHD_PBF, U12 LTC3130, U13 LTC4376CDHD_PBF, U14 SI3865DDV-T1-GE3, U2 ADM1176-1ARMZ-R7, U3 LTC3130, U4 LTC3130, U5 DRV8830DRC, U6 ADM1176-1ARMZ-R7, U7 SI3865DDV-T1-GE3, U8 LTC4376CDHD_PBF, U9 SI3865DDV-T1-GE3

Commit message: v1 Final
Parts:
- moved ? 15.7 mm to (158.2, 43.7)
- moved REF** 15.7 mm to (162.4, 46.7)
Changed lines of the file:
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@@
 			(drillshape 0)
 			(scaleselection 1)
-			(outputdirectory "../Gerbers2_0.8/")
+			(outputdirectory "../../Gerbers/SolarPanels/")
 		)
 	)
@@
 	(footprint "clipboard:eb50a26b-5fb6-463a-8dd0-ee5887daaa13"
 		(layer "F.Cu")
-		(at 148.256812 55.861755)
+		(at 158.2168 43.720555)
 		(property "Reference" ""
 			(at 0 0 0)
@@
 	(footprint "X Label"
 		(layer "F.Cu")
-		(at 152.396812 58.8772)
+		(at 162.3568 46.736)
 		(property "Reference" "REF**"
 			(at 0 -12.2 0)
@@
 		(tags "resistor")
 		(property "Reference" "R76"
-			(at 0.012201 -10.3378 90)
+			(at 0.2416 5.5118 90)
 			(layer "B.SilkS")
 			(effects
@@
 		(tags "resistor")
 		(property "Reference" "R81"
-			(at 0.013298 10.3434 90)
+			(at 0.215699 5.492 90)
 			(layer "B.SilkS")
 			(effects
@@
 		(tags "SOT-363 SC-70-6")
 		(property "Reference" "Q16"
-			(at -6.8458 -1.587002 0)
+			(at -2.1976 -0.825801 90)
 			(layer "B.SilkS")
 			(effects
@@
 		(layer "B.SilkS")
 	)
+	(gr_rect
+		(start 149.4282 54.4068)
+		(end 155.3718 60.1218)
+		(stroke
+			(width 0.0254)
+			(type solid)
+		)
+		(fill solid)
+		(layer "F.SilkS")
+	)
 	(gr_line
