File: DeploymentSensor.kicad_sch (KiCad schematic)
At the start: 5 parts, among them U11 VL53L4CX

Commit message: Local Stash
Parts:
- U11: value VL53L4CX -> VL53L4CD
Changed lines of the file:
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@@
 			)
 		)
-		(property "Value" "VL53L4CX"
+		(property "Value" "VL53L4CD"
 			(at 120.396 117.094 0)
 			(effects

Commit message: V4 Updates and Cell Backer
Other:
- title: (none) -> Argus XY Solar Panel
Changed lines of the file:
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@@
 	(paper "A4")
 	(title_block
-		(date "2025-04-20")
-		(rev "v3.1")
+		(title "Argus XY Solar Panel")
+		(date "2026-01-27")
+		(rev "v4.0")
 		(company "Carnegie Mellon University")
 		(comment 1 "N. Khera")
