File: XY/Avionics-SolarPanels.kicad_sch (KiCad schematic)
At the start: 37 parts, among them J1 200528-0100, J2 200528-0100

Commit message: Z- Board Files
Parts:
- R10, R18, R5: value R_Small -> 107K
- R12, R20, R7: value R_Small -> 1.47M
- R13, R21, R8: value R_Small -> 200K
- R17, R3, R9: value R_Small -> 1.91M
Changed lines of the file:
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@@
 			)
 		)
-		(property "Value" "R_Small"
-			(at 35.052 176.276 0)
+		(property "Value" "107K"
+			(at 37.846 176.276 0)
 			(effects
 				(font
@@
 			)
 		)
-		(property "Value" "R_Small"
-			(at 103.378 87.376 0)
+		(property "Value" "200K"
+			(at 100.838 87.376 0)
 			(effects
 				(font
@@
 			)
 		)
-		(property "Value" "R_Small"
-			(at 103.378 168.656 0)
+		(property "Value" "1.47M"
+			(at 101.6 168.656 0)
 			(effects
 				(font
@@
 			)
 		)
-		(property "Value" "R_Small"
-			(at 35.052 168.656 0)
+		(property "Value" "1.91M"
+			(at 37.084 168.656 0)
 			(effects
 				(font
@@
 			)
 		)
-		(property "Value" "R_Small"
-			(at 103.378 131.826 0)
+		(property "Value" "200K"
+			(at 100.838 131.826 0)
 			(effects
 				(font
@@
 			)
 		)
-		(property "Value" "R_Small"
-			(at 103.378 176.276 0)
+		(property "Value" "200K"
+			(at 100.584 176.276 0)
 			(effects
 				(font
@@
 			)
 		)
-		(property "Value" "R_Small"
-			(at 35.052 131.826 0)
+		(property "Value" "107K"
+			(at 37.846 131.826 0)
 			(effects
 				(font
@@
 			)
 		)
-		(property "Value" "R_Small"
-			(at 103.378 79.756 0)
+		(property "Value" "1.47M"
+			(at 101.6 79.756 0)
 			(effects
 				(font
@@
 			)
 		)
-		(property "Value" "R_Small"
-			(at 103.378 124.206 0)
+		(property "Value" "1.47M"
+			(at 101.6 124.206 0)
 			(effects
 				(font
@@
 			)
 		)
-		(property "Value" "R_Small"
-			(at 35.052 124.206 0)
+		(property "Value" "1.91M"
+			(at 37.084 124.206 0)
 			(effects
 				(font
@@
 			)
 		)
-		(property "Value" "R_Small"
-			(at 35.052 87.376 0)
+		(property "Value" "107K"
+			(at 37.846 87.376 0)
 			(effects
 				(font
@@
 			)
 		)
-		(property "Value" "R_Small"
-			(at 35.052 79.756 0)
-			(effects
-				(font
+		(property "Value" "1.91M"
+			(at 37.084 79.756 0)
+			(effects
+				(font

Commit message: MPPT fixes
Parts:
- added R108, R111, R113: 127k, Resistor_SMD:R_0603_1608Metric, symbol Device:R_Small
- added R109, R110, R112: 1.91M, Resistor_SMD:R_0603_1608Metric, symbol Device:R_Small
Connections:
- net D_VSOLAR1: now also R110.1
- net D_VSOLAR2: now also R112.1
- net GND: now also R108.2, R111.2, R113.2
- net VSOLAR: now also R109.1
- new net MPPT/RUN: R108.1, R109.2
- new net MPPT1/RUN: R110.2, R111.1
- new net MPPT2/RUN: R112.2, R113.1
Other:
- sheet Charge OR-ing ports: added none; removed PGOOD
- sheet Charge OR-ing1 ports: added none; removed PGOOD
- sheet Charge OR-ing2 ports: added none; removed PGOOD
- sheet MPPT ports: added RUN; removed none
- sheet MPPT1 ports: added RUN; removed none
- sheet MPPT2 ports: added RUN; removed none
