File: XY/Avionics-SolarPanels.kicad_sch (KiCad schematic)
At the start: 6 parts

Commit message: almost done
Parts:
- H1, H2, H3, H4: footprint SolarPanels:MountingHole_3.2mm_M3_DIN965_Pad_TopBottom -> MountingHole:MountingHole_3.2mm_M3_DIN965_Pad_TopBottom
- H5, H6: footprint SolarPanels:MountingHole_3mm -> MountingHole:MountingHole_3mm
Changed lines of the file:
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@@
 			)
 		)
-		(property "Footprint" "SolarPanels:MountingHole_3.2mm_M3_DIN965_Pad_TopBottom"
+		(property "Footprint" "MountingHole:MountingHole_3.2mm_M3_DIN965_Pad_TopBottom"
 			(at 170.18 53.34 0)
 			(effects
@@
 			)
 		)
-		(property "Footprint" "SolarPanels:MountingHole_3mm"
+		(property "Footprint" "MountingHole:MountingHole_3mm"
 			(at 170.18 119.38 0)
 			(effects
@@
 			)
 		)
-		(property "Footprint" "SolarPanels:MountingHole_3.2mm_M3_DIN965_Pad_TopBottom"
+		(property "Footprint" "MountingHole:MountingHole_3.2mm_M3_DIN965_Pad_TopBottom"
 			(at 170.18 83.82 0)
 			(effects
@@
 			)
 		)
-		(property "Footprint" "SolarPanels:MountingHole_3mm"
+		(property "Footprint" "MountingHole:MountingHole_3mm"
 			(at 170.18 129.54 0)
 			(effects
@@
 			)
 		)
-		(property "Footprint" "SolarPanels:MountingHole_3.2mm_M3_DIN965_Pad_TopBottom"
+		(property "Footprint" "MountingHole:MountingHole_3.2mm_M3_DIN965_Pad_TopBottom"
 			(at 170.18 63.5 0)
 			(effects
@@
 			)
 		)
-		(property "Footprint" "SolarPanels:MountingHole_3.2mm_M3_DIN965_Pad_TopBottom"
+		(property "Footprint" "MountingHole:MountingHole_3.2mm_M3_DIN965_Pad_TopBottom"
 			(at 170.18 73.66 0)
 			(effects

Commit message: Uncommitted schematic changes
Parts:
- H5, H6: footprint MountingHole:MountingHole_3mm -> MountingHole:MountingHole_3mm_Pad_TopBottom
Changed lines of the file:
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@@
 			)
 		)
-		(property "Footprint" "MountingHole:MountingHole_3mm"
+		(property "Footprint" "MountingHole:MountingHole_3mm_Pad_TopBottom"
 			(at 170.18 119.38 0)
 			(effects
@@
 			)
 		)
-		(property "Footprint" "MountingHole:MountingHole_3mm"
+		(property "Footprint" "MountingHole:MountingHole_3mm_Pad_TopBottom"
 			(at 170.18 129.54 0)
 			(effects
