File: XY/MPPT.kicad_sch (KiCad schematic)
At the start: 15 parts, among them U4 LTC3130

Commit message: MPPT fixes
Connections:
- net VIN: no longer U4.4 (RUN)
- new net RUN: U4.4 (RUN)
Changed lines of the file:
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@@
-	)
-	(junction
-		(at 128.905 92.71)
-		(diameter 0)
-		(color 0 0 0 0)
 	)
 	(junction
@@
 	(wire
 		(pts
-			(xy 128.905 92.71) (xy 128.905 97.79)
-		)
-		(stroke
-			(width 0)
-			(type default)
-		)
-	)
-	(wire
-		(pts
 			(xy 146.685 68.58) (xy 149.225 68.58)
 		)
@@
 	(wire
 		(pts
-			(xy 89.535 92.71) (xy 128.905 92.71)
-		)
-		(stroke
-			(width 0)
-			(type default)
-		)
-	)
-	(wire
-		(pts
 			(xy 89.535 128.27) (xy 118.11 128.27)
 		)
@@
 	(wire
 		(pts
+			(xy 102.87 97.79) (xy 132.08 97.79)
+		)
+		(stroke
+			(width 0)
+			(type default)
+		)
+	)
+	(wire
+		(pts
 			(xy 58.42 90.17) (xy 58.42 93.98)
 		)
@@
 	(wire
 		(pts
-			(xy 128.905 92.71) (xy 132.08 92.71)
+			(xy 89.535 92.71) (xy 132.08 92.71)
 		)
 		(stroke
@@
 		(pts
 			(xy 118.11 107.95) (xy 118.11 116.84)
-		)
-		(stroke
-			(width 0)
-			(type default)
-		)
-	)
-	(wire
-		(pts
-			(xy 128.905 97.79) (xy 132.08 97.79)
 		)
 		(stroke
@@
 		)
 	)
+	(hierarchical_label "RUN"
+		(shape output)
+		(at 102.87 97.79 180)
+		(fields_autoplaced yes)
+		(effects
+			(font
+				(size 1.27 1.27)
+			)
+			(justify right)
+		)
+	)
