File: XY/MPPT.kicad_sch (KiCad schematic)
At the start: 15 parts, among them U10 LTC3130

Commit message: almost done
Parts:
- U10: symbol SolarPanels:LTC3130 -> Argus-IC:LTC3130
Changed lines of the file:
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@@
 	)
 	(symbol
-		(lib_id "SolarPanels:LTC3130")
+		(lib_id "Argus-IC:LTC3130")
 		(at 153.67 102.87 0)
 		(unit 1)

Commit message: Updated 3d models, footprints
Parts:
- L1: footprint Inductor_SMD:L_Coilcraft_LPS4018 -> Argus-Passives:L_Coilcraft_LPS4018
Changed lines of the file:
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@@
 			)
 		)
-		(property "Footprint" "Inductor_SMD:L_Coilcraft_LPS4018"
+		(property "Footprint" "Argus-Passives:L_Coilcraft_LPS4018"
 			(at 153.035 68.58 0)
 			(effects
