File: XY/LightSensor.kicad_sch (KiCad schematic)
At the start: 7 parts, among them U5 OPT4003DNPRQ1

Commit message: Updated layout
Parts:
- F1: footprint (none) -> Fuse:Fuse_0603_1608Metric
Changed lines of the file:
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@@
 			)
 		)
-		(property "Footprint" ""
+		(property "Footprint" "Fuse:Fuse_0603_1608Metric"
 			(at 116.84 82.55 0)
 			(effects

Commit message: almost done
Parts:
- U5: symbol SolarPanels:OPT4003DNPRQ1 -> Argus-IC:OPT4003DNPRQ1
Changed lines of the file:
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@@
 	)
 	(symbol
-		(lib_id "SolarPanels:OPT4003DNPRQ1")
+		(lib_id "Argus-IC:OPT4003DNPRQ1")
 		(at 142.24 100.33 0)
 		(unit 1)

Commit message: Uncommitted schematic changes
Parts:
- U5: footprint SolarPanels:OPT4003 -> Argus-IC:OPT4003
Changed lines of the file:
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@@
 			)
 		)
-		(property "Footprint" "SolarPanels:OPT4003"
+		(property "Footprint" "Argus-IC:OPT4003"
 			(at 129.794 112.014 0)
 			(effects
