File: Z+/CoilDriver.kicad_sch (KiCad schematic)
At the start: 27 parts, among them Q20 IRLML2803, Q21 SiRA99DP, U2 DRV8235RTER

Commit message: Z+ updates WIP
Parts:
- R33: renamed from R88; symbol SolarPanels:R_Small -> Device:R_Small
- renumbered C15 to C12, C16 to C13, C17 to C14, D7 to D3, D8 to D4, F2 to F6, Q20 to Q8, Q21 to Q9, R68 to R19, R69 to R20, R70 to R21, R77 to R22, R78 to R23, R79 to R24, R80 to R25, R81 to R26, R82 to R27, R83 to R28, R84 to R29, R85 to R30, R86 to R31, R87 to R32, R89 to R34, R90 to R35, U2 to U7
