File: Z+/I2CSingleProtection.kicad_sch (KiCad schematic)
At the start: 10 parts, among them Q19 NX3008NBKS, Q25 MBT2222ADW1T1, Q26 MBT2222ADW1T1

Commit message: Z+ updates WIP
Parts:
- renumbered C42 to C27, Q19 to Q14, Q26 to Q15, Q25 to Q15, R107 to R62, R108 to R63, R109 to R64, R110 to R65, R111 to R66, R112 to R67
