File: Z+/Z+.kicad_pcb (KiCad board)
At the start: 4 copper layers, 98 x 98 mm, 222 parts, among them J1 200528-0100, J2 Conn_01x04_MountingPin, J3 USB4110GFA, J4 BG301-06-X-XXXX-X-X_REVC, J5 BG301-06-X-XXXX-X-X_REVC, Q1 NX3008NBKS, Q10 NX3008NBKS, Q11 MBT2222ADW1T1, Q12 NX3008NBKS, Q13 MBT2222ADW1T1, Q14 NX3008NBKS, Q15 MBT2222ADW1T1, Q16 NX3008NBKS, Q17 MBT2222ADW1T1, Q18 NX3008NBKS, Q19 MBT2222ADW1T1, Q2 MBT2222ADW1T1, Q20 NX3008NBKS, Q21 MBT2222ADW1T1, Q22 NX3008NBKS, Q23 MBT2222ADW1T1, Q24 NX3008NBKS, Q25 MBT2222ADW1T1, Q26 NX3008NBKS, Q27 MBT2222ADW1T1, Q3 NX3008NBKS, Q4 MBT2222ADW1T1, Q5 NX3008NBKS, Q6 MBT2222ADW1T1, Q7 SiRA99DP, Q8 IRLML2803, Q9 SiRA99DP, U1 USBLC6-2P6, U10 USBLC6-2P6, U2 SunSensor, U3 SunSensor, U4 SunSensor, U5 SunSensor, U6 LTC4412xS6, U7 DRV8235RTER, U8 ADM1176-1ARMZ-R7, U9 LTC3130

Commit message: Finished layout v1
Parts:
- removed D1: ESD5Zxx, Diode_SMD:D_SOD-523
- added R113: 0R, Resistor_SMD:R_0603_1608Metric, B.Cu at (172.2, 84.1)
- added R114: 0R, Resistor_SMD:R_0603_1608Metric, B.Cu at (172.2, 82.3)
- added R115: 0R, Resistor_SMD:R_0603_1608Metric, B.Cu at (174.0, 82.3)
- added R116: 0R, Resistor_SMD:R_0603_1608Metric, B.Cu at (174.0, 84.1)
- moved C2 3.33 mm to (175.6, 84.1), turned to -90 degrees
- moved C1 3.14 mm to (169.2, 84.1), turned to -90 degrees
Connections:
- J1 pad 3: COIL_DRIVER_EN -> /Interfaces/COIL_DRIVER_EN_OR_MAIN_3V3
- J1 pad 5: PERI_3V3 -> /Interfaces/PERI_3V3_OR_GND
Routing:
- net PERI_3V3: track 0.00 -> 335.5 mm, vias 0 -> 6
- net SDA: track 22.8 -> 144.8 mm, vias 0 -> 7
- net SCL: track 26.6 -> 136.0 mm, vias 0 -> 7
- net VBATT: track 30.3 -> 94.8 mm, vias 1 -> 5
- net /Sun Pyramid/LS3_3V3: track 7.09 -> 63.5 mm, vias 0 -> 3
- net Net-(D10-A): track 34.2 -> 81.4 mm
- net COIL_DRIVER_EN: track 0.00 -> 43.5 mm, vias 0 -> 2
- net MAIN_3V3: track 1.52 -> 42.1 mm, vias 0 -> 11
- net VSOLAR: track 22.1 -> 49.4 mm, vias 0 -> 2
- net /Coil Driver/SCL_M: track 14.9 -> 39.4 mm, vias 1 -> 2
- net /Coil Driver/SDA_M: track 14.8 -> 36.3 mm, vias 1 -> 2
- net SDA_SPWR: track 10.1 -> 28.7 mm, vias 0 -> 2
- net SCL_SPWR: track 10.1 -> 24.3 mm
- net /Interfaces/COIL_DRIVER_EN_OR_MAIN_3V3: track 0.00 -> 8.45 mm
- net /Interfaces/PERI_3V3_OR_GND: track 0.00 -> 4.93 mm
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- added copper zone on B.Cu, net /Coil Driver/VM
- added copper zone on In1.Cu, net MAIN_3V3
- added copper zone on B.Cu, net VBATT
- added copper zone on B.Cu, net VSOLAR
- removed copper zone on In1.Cu, net COIL_DRIVER_EN
